File: dap42.kicad_pcb (KiCad board)
At the start: 2 copper layers, 35 x 15 mm, 33 parts, among them J1 USB_B_Micro, J2 Conn_02x05_Odd_Even, J4 Conn_01x04, SW1 SW_SPST, U1 WE-TVS-82400102, U2 SPX3819M5-L-3-3, U3 STM32F102C8Tx

Commit message: Add crystal
Parts:
- added C11: 20pF, Capacitor_SMD:C_0402_1005Metric_Pad0.74x0.62mm_HandSolder, F.Cu at (157.3, 98.2)
- added C12: 20pF, Capacitor_SMD:C_0402_1005Metric_Pad0.74x0.62mm_HandSolder, F.Cu at (157.3, 93.7)
- added R13: 1M 0402, Resistor_SMD:R_0402_1005Metric_Pad0.72x0.64mm_HandSolder, F.Cu at (157.3, 95.9)
- added Y1: 8MHz, Crystal:Crystal_HC49-U_Vertical, F.Cu at (154.0, 97.7)
- C1: value 1uF 0603 -> 1uF 0402; footprint Capacitor_SMD:C_0603_1608Metric_Pad1.08x0.95mm_HandSolder -> Capacitor_SMD:C_0402_1005Metric_Pad0.74x0.62mm_HandSolder
- C2: value 4.7uF 0603 -> 4.7uF 0402; footprint Capacitor_SMD:C_0603_1608Metric_Pad1.08x0.95mm_HandSolder -> Capacitor_SMD:C_0402_1005Metric_Pad0.74x0.62mm_HandSolder
- C5: value 0.1uF 0402 -> 0.1uF
- D3: value LED_GBAR -> LED_ARGB; footprint dap42:B38G3RGB -> dap42:XZCMEDGCBD110W
- R3: value 4.7k 0603 -> 10k 0402; footprint Resistor_SMD:R_0603_1608Metric_Pad0.98x0.95mm_HandSolder -> Resistor_SMD:R_0402_1005Metric_Pad0.72x0.64mm_HandSolder
- R6, R7: value 1k 0402 -> 100 0402
- R8: value 1k 0402 -> 200 0402
- R9: value 10k 0402 -> 10k
- moved R1 5.14 mm to (152.9, 88.4)
- moved J2 5.04 mm to (148.0, 95.0)
- moved R11 4.60 mm to (152.3, 101.8), turned to 0 degrees
- moved C7 4.47 mm to (158.1, 100.6), turned to 180 degrees
- moved C10 3.87 mm to (154.6, 101.8), turned to 180 degrees
- moved R3 3.35 mm to (177.2, 93.4)
- moved C3 3.13 mm to (170.7, 99.6), turned to -90 degrees
- moved C1 2.70 mm to (155.7, 88.7), turned to 0 degrees
- moved D3 2.62 mm to (158.4, 88.8), turned to 180 degrees
- moved R8 2.44 mm to (161.0, 89.3)
- moved R10 0.89 mm to (158.6, 101.7), turned to 0 degrees
- moved C9 0.38 mm to (158.7, 92.0)
- moved U1 0.23 mm to (177.2, 95.7)
Connections:
- D3 pad 1: Net-(R7-Pad2) -> +3V3
- D3 pad 2: Net-(R6-Pad2) -> Net-(D3-Pad2)
- D3 pad 3: +3V3 -> Net-(D3-Pad3)
- D3 pad 4: Net-(R8-Pad2) -> Net-(D3-Pad4)
- R10 pad 1: Net-(R10-Pad1) -> /~{RESET}
- R10 pad 2: /~{RESET} -> Net-(R10-Pad2)
- R6 pad 1: Net-(R6-Pad1) -> /LEDB
- R6 pad 2: Net-(R6-Pad2) -> Net-(D3-Pad4)
- R7 pad 1: Net-(R7-Pad1) -> /LEDG
- R7 pad 2: Net-(R7-Pad2) -> Net-(D3-Pad3)
- R8 pad 1: Net-(R8-Pad1) -> /LEDR
- R8 pad 2: Net-(R8-Pad2) -> Net-(D3-Pad2)
- U3 pad 12: unconnected-(U3-Pad12) -> /TX
- U3 pad 13: unconnected-(U3-Pad13) -> /RX
- U3 pad 15: Net-(R10-Pad1) -> unconnected-(U3-Pad15)
- U3 pad 18: unconnected-(U3-Pad18) -> Net-(R10-Pad2)
- U3 pad 2: unconnected-(U3-Pad2) -> /LEDB
- U3 pad 25: unconnected-(U3-Pad25) -> /TDI
- U3 pad 26: unconnected-(U3-Pad26) -> /SWCLK/TCK
- U3 pad 27: unconnected-(U3-Pad27) -> /SWDIO/TMS
- U3 pad 28: /SWDIO/TMS -> /SWO/TDO
- U3 pad 29: /SWCLK/TCK -> unconnected-(U3-Pad29)
- U3 pad 3: unconnected-(U3-Pad3) -> /LEDR
- U3 pad 30: /TDI -> unconnected-(U3-Pad30)
- U3 pad 31: /SWO/TDO -> unconnected-(U3-Pad31)
- U3 pad 4: unconnected-(U3-Pad4) -> /LEDG
- U3 pad 41: Net-(R6-Pad1) -> unconnected-(U3-Pad41)
- U3 pad 43: Net-(R7-Pad1) -> unconnected-(U3-Pad43)
- U3 pad 46: Net-(R8-Pad1) -> unconnected-(U3-Pad46)
- U3 pad 5: unconnected-(U3-Pad5) -> /OSCIN
- U3 pad 6: unconnected-(U3-Pad6) -> /OSCOUT
Routing:
- net /~{RESET}: track 6.22 -> 21.7 mm, vias 0 -> 2
- net Net-(R8-Pad1): track 14.1 -> 0.00 mm, vias 2 -> 0
- net /TDI: track 15.2 -> 29.2 mm, vias 1 -> 2
- net /SWO/TDO: track 15.3 -> 29.4 mm, vias 1 -> 2
- net /LEDG: track 0.00 -> 11.5 mm, vias 0 -> 2
- net Net-(R7-Pad1): track 11.4 -> 0.00 mm, vias 2 -> 0
- net /SWDIO/TMS: track 19.5 -> 30.1 mm, vias 1 -> 2
- net /SWCLK/TCK: track 18.8 -> 29.4 mm, vias 1 -> 2
- net /LEDR: track 0.00 -> 8.62 mm, vias 0 -> 2
- net /LEDB: track 0.00 -> 8.36 mm, vias 0 -> 2
- net Net-(R6-Pad1): track 7.27 -> 0.00 mm, vias 2 -> 0
- net /OSCIN: track 0.00 -> 7.17 mm
- net /OSCOUT: track 0.00 -> 6.48 mm
- net Net-(D3-Pad3): track 0.00 -> 5.48 mm
- net Net-(R10-Pad2): track 0.00 -> 4.52 mm
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Other:
- board size 35 x 15 mm -> 40 x 15 mm
- board text added: "DAP42 STM32F103C8 v2 PSYONIC Jonathan Mullen"
- board text removed: "DAP42 STM32F103C8 v1.0 PSYONIC Jonathan Mullen"
