File: dap42.kicad_sch (KiCad schematic)
At the start: 33 parts, among them J1 USB_B_Micro, J2 Conn_02x05_Odd_Even, J4 Conn_01x04, SW1 SW_SPST, U1 WE-TVS-82400102, U2 SPX3819M5-L-3-3, U3 STM32F102C8Tx

Commit message: Add crystal
Parts:
- added C11, C12: 20pF, Capacitor_SMD:C_0402_1005Metric_Pad0.74x0.62mm_HandSolder, symbol Device:C
- added R13: 1M 0402, Resistor_SMD:R_0402_1005Metric_Pad0.72x0.64mm_HandSolder, symbol Device:R_US
- added Y1: 8MHz, Crystal:Crystal_HC49-U_Vertical, symbol Device:Crystal
- C1: value 1uF 0603 -> 1uF 0402; footprint Capacitor_SMD:C_0603_1608Metric_Pad1.08x0.95mm_HandSolder -> Capacitor_SMD:C_0402_1005Metric_Pad0.74x0.62mm_HandSolder
- C2: value 4.7uF 0603 -> 4.7uF 0402; footprint Capacitor_SMD:C_0603_1608Metric_Pad1.08x0.95mm_HandSolder -> Capacitor_SMD:C_0402_1005Metric_Pad0.74x0.62mm_HandSolder
- C5: value 0.1uF 0402 -> 0.1uF
- D3: value LED_GBAR -> LED_ARGB; footprint dap42:B38G3RGB -> dap42:XZCMEDGCBD110W; symbol Device:LED_GBAR -> Device:LED_ARGB; MPN (none) -> XZCMEDGCBD110W
- R3: value 4.7k 0603 -> 10k 0402; footprint Resistor_SMD:R_0603_1608Metric_Pad0.98x0.95mm_HandSolder -> Resistor_SMD:R_0402_1005Metric_Pad0.72x0.64mm_HandSolder
- R6, R7: value 1k 0402 -> 100 0402
- R8: value 1k 0402 -> 200 0402
- R9: value 10k 0402 -> 10k
Connections:
- net +3V3: now also D3.1 (A); no longer D3.3 (A)
- net GND: now also C11.2, C12.2
- net SWCLK/TCK: now also U3.26 (PB13); no longer U3.29 (PA8)
- net SWDIO/TMS: now also U3.27 (PB14); no longer U3.28 (PB15)
- net SWO/TDO: now also U3.28 (PB15); no longer U3.31 (PA10)
- net TDI: now also U3.25 (PB12); no longer U3.30 (PA9)
- net ~{RESET}: now also R10.1; no longer R10.2
- net at R7.2: now also D3.3 (GK); no longer D3.1 (GK)
- net at D3.2 (RK): now also R8.2; no longer R6.2
- net at D3.4 (BK): now also R6.2; no longer R8.2
- net TX: now reaches U3.12 (PA2)
- net RX: now reaches U3.13 (PA3)
- net at U3.15 (PA5): no longer R10.1
- net at U3.18 (PB0): now also R10.2
- net LEDB: now reaches U3.2 (PC13)
- net LEDB: now also R6.1
- net LEDR: now reaches U3.3 (PC14)
- net LEDR: now also R8.1
- net LEDG: now reaches U3.4 (PC15)
- net LEDG: now also R7.1
- net at U3.41 (PB5): no longer R6.1
- net at U3.43 (PB7): no longer R7.1
- net at U3.46 (PB9): no longer R8.1
- net OSCIN: now reaches U3.5 (PD0)
- net OSCIN: now also C12.1, R13.1, Y1.2
- net OSCOUT: now reaches U3.6 (PD1)
- net OSCOUT: now also C11.1, R13.2, Y1.1
- no-connect marks 28 -> 24
Other:
- moved on the sheet: D3, R10, R11, R6, R7, R8
